File: RHS_3.kicad_pcb (KiCad board)
At the start: 2 copper layers, 51 x 61 mm, 35 parts, among them IC1 ATMEGA328P-A, IC2 CC1101, P4 ISP Bottom, P5 ISP Top, P6 FTDI, P7 ISP 10, SW1 Reset, SW2 Config, U1 TLE4913, U2 TLE4913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

Commit message: v1.1
Parts:
- removed JP1, JP2: SolderJumper_3_Open, Jumper:SolderJumper-3_P1.3mm_Open_Pad1.0x1.5mm_NumberLabels
- added C13: 10p, Capacitor_SMD:C_0805_2012Metric_Pad1.15x1.40mm_HandSolder, B.Cu at (69.4, 121.9)
- added J1: Glass Breakage Detector, TerminalBlock:TerminalBlock_bornier-2_P5.08mm, F.Cu at (73.5, 126.9)
- added J2: ANT, Connector_Pin:Pin_D1.0mm_L10.0mm, F.Cu at (69.1, 72.1)
- added R7: 1M, Resistor_SMD:R_0805_2012Metric_Pad1.15x1.40mm_HandSolder, B.Cu at (67.2, 121.8)
- C1, C10, C11, C12, C2, C3, C4, C5, C6, C7, C8, C9, IC1, IC2, R1, R2, R3, R4, R5, R6, U1, U2, U3, Y1: moved to B.Cu
- moved D2 53.9 mm to (65.2, 73.5)
- moved SW2 53.0 mm to (63.4, 79.5), turned to 270 degrees
- moved D1 49.9 mm to (63.2, 73.5), turned to 270 degrees
- moved IC2 35.8 mm to (70.1, 84.1)
- moved C12 26.5 mm to (63.6, 107.7), turned to 180 degrees
- moved C1 25.8 mm to (67.2, 111.4), turned to 270 degrees
- moved SW1 22.2 mm to (63.4, 119.8), turned to 270 degrees
- moved Y1 21.9 mm to (67.2, 107.0), turned to 270 degrees
- moved R3 19.8 mm to (69.4, 101.7), turned to 270 degrees
- moved C11 19.8 mm to (63.5, 110.1), turned to 180 degrees
- moved C7 17.6 mm to (77.2, 116.4), turned to 180 degrees
- moved P7 17.4 mm to (90.5, 79.3), turned to 270 degrees
- moved R2 15.5 mm to (67.2, 101.6), turned to 270 degrees
- moved P6 14.9 mm to (87.5, 106.5)
- moved IC1 14.1 mm to (74.6, 109.0)
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Connections:
- R4 pad 1: Net-(JP2-Pad2) -> VCC
- R5 pad 1: Net-(JP2-Pad2) -> VCC
- R6 pad 1: Net-(JP1-Pad2) -> VCC
Routing:
- net /MISO: track 99.2 -> 50.8 mm, vias 3 -> 2
- net /SCK: track 97.2 -> 50.9 mm, vias 4 -> 2
- net Net-(JP2-Pad2): track 35.5 -> 0.00 mm
- net /D6: track 32.8 -> 0.00 mm, vias 2 -> 0
- net /MOSI: track 84.2 -> 53.3 mm, vias 4 -> 0
- net Net-(IC1-Pad12): track 7.60 -> 36.0 mm, vias 0 -> 1
- net VCC: track 165.1 -> 193.3 mm, vias 4 -> 5
- net Net-(D2-Pad2): track 9.42 -> 33.9 mm, vias 0 -> 1
- net Net-(IC1-Pad14): track 44.1 -> 19.9 mm, vias 2 -> 0
- net Net-(IC1-Pad9): track 27.7 -> 4.44 mm, vias 2 -> 0
- net Net-(D1-Pad2): track 8.95 -> 31.4 mm, vias 0 -> 1
- net /A2: track 39.3 -> 28.2 mm
- net /RXD: track 43.7 -> 54.8 mm
- net /A1: track 33.0 -> 43.5 mm
- net /TXD: track 46.7 -> 56.3 mm, vias 2 -> 1
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Other:
- board text added: "Glass Breakage Detector"
- board text added: "RHS-3 V1.1"

Commit message: V1.1 ready
Parts:
- J1: footprint TerminalBlock:TerminalBlock_bornier-2_P5.08mm -> Connector_JST:JST_XH_S2B-XH-A-1_1x02_P2.50mm_Horizontal
- moved R7 5.46 mm to (72.6, 121.8)
- moved C13 5.39 mm to (74.8, 121.8), turned to 270 degrees
- moved J1 4.49 mm to (70.0, 124.2)
Routing:
- net /A3: track 24.7 -> 16.9 mm
- net VCC: track 193.3 -> 189.5 mm
- net /RESET: track 67.7 -> 68.7 mm
