File: RHS_3.kicad_pcb (KiCad board)
At the start: 2 copper layers, 51 x 61 mm, 68 parts, among them IC1 ATMEGA328P-A, IC2 CC1101, IC3 CC1101_Chip, J1 Glass Breakage Detector, J2 ANT, P4 ISP Bottom, P5 ISP Top, P6 FTDI, P7 ISP 10, Q1 Si2305CDS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

Commit message: gerber and production files updated
Parts:
- moved R8 0.91 mm to (76.9, 86.4)
- moved C22 0.70 mm to (68.3, 90.3), turned to 270 degrees
- moved C20 0.44 mm to (70.4, 90.2)
Routing:
- net VDC: track 65.0 -> 63.6 mm
- net GND: track 86.4 -> 85.0 mm, vias 38 -> 37
- net Net-(IC3-Pad17): track 4.30 -> 3.26 mm

Commit message: fix 100p
Parts:
- C27: value 100n -> 100p
Changed lines of the file:
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@@
       (effects (font (size 1 1) (thickness 0.15)) (justify mirror))
     )
-    (fp_text value 100n (at 0 -1.17 90) (layer B.Fab) hide
+    (fp_text value 100p (at 0 -1.17 90) (layer B.Fab) hide
       (effects (font (size 1 1) (thickness 0.15)) (justify mirror))
     )
