File: RHS_3_Simple.kicad_pcb (KiCad board)
At the start: 2 copper layers, 21 x 100.5 mm, 37 parts, among them IC1 ATMEGA328P-A, IC2 CC1101, J1 Glass Breakage Detector, J2 ANT, P4 ISP Bottom, P5 ISP Top, P6 FTDI, P7 ISP 10, SW1 Reset, SW2 Config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

Commit message: alternative pcb layout
Parts:
- C10, C6, R2, R3, R6, U3: moved to F.Cu
- moved J1 45.7 mm to (104.1, 133.0), turned to 180 degrees
- moved R7 43.0 mm to (101.6, 135.9), turned to 0 degrees
- moved C13 40.1 mm to (101.6, 137.9), turned to 180 degrees
- moved C10 28.3 mm to (91.9, 138.0)
- moved C6 28.2 mm to (92.0, 145.8)
- moved R6 27.5 mm to (92.0, 140.1)
- moved U3 27.2 mm to (91.9, 142.9), turned to 270 degrees
- moved P4 24.2 mm to (94.0, 130.3), turned to 90 degrees
- moved P5 24.1 mm to (94.0, 130.3), turned to 270 degrees
- moved SW1 11.8 mm to (92.0, 178.5)
- moved J2 10.5 mm to (108.0, 179.0)
- moved BT1 10.5 mm to (100.0, 161.5)
- moved IC2 9.85 mm to (100.0, 168.0)
- moved C3 9.52 mm to (94.0, 155.0), turned to 0 degrees
- moved SW2 9.40 mm to (101.0, 138.4), turned to 0 degrees
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Other:
- board size 21 x 100.5 mm -> 21 x 99.5 mm

Commit message: V1.1 ready
Parts:
- J1: footprint TerminalBlock:TerminalBlock_bornier-2_P5.08mm -> Connector_PinHeader_2.00mm:PinHeader_2x01_P2.00mm_Vertical_SMD
- P7: footprint Connector_PinHeader_2.54mm:PinHeader_2x05_P2.54mm_Vertical -> Connector_PinHeader_2.00mm:PinHeader_2x05_P2.00mm_Vertical_SMD
- R2, R3: moved to B.Cu
- moved SW2 41.3 mm to (107.8, 179.2), turned to 90 degrees
- moved P7 25.5 mm to (100.7, 138.4)
- moved J1 6.88 mm to (108.3, 138.4), turned to 270 degrees
- moved D1 6.48 mm to (106.7, 145.4), turned to 90 degrees
- moved D2 6.48 mm to (108.7, 145.4), turned to 90 degrees
- moved J2 5.70 mm to (108.8, 173.4)
- moved R3 2.29 mm to (108.7, 141.0), turned to 90 degrees
- moved R2 2.29 mm to (106.7, 141.0), turned to 90 degrees
- moved SW1 0.57 mm to (92.0, 179.1)

Commit message: small version layouted
Parts:
- removed C7: 100n, Capacitor_SMD:C_0805_2012Metric_Pad1.15x1.40mm_HandSolder
- removed P6: FTDI, Connector_PinHeader_2.54mm:PinHeader_1x06_P2.54mm_Vertical
- moved C6 0.77 mm to (91.9, 146.6)
- moved C11 0.51 mm to (108.5, 147.3)
- moved C12 0.51 mm to (108.5, 151.9)
- moved U3 0.44 mm to (91.9, 143.4)
- moved C10 0.41 mm to (91.9, 138.4)
- moved R6 0.35 mm to (91.9, 140.5)
- moved R3 0.25 mm to (108.5, 141.0)
- moved C13 0.25 mm to (101.6, 137.7)
- moved R7 0.25 mm to (101.6, 135.6)
- moved Y1 0.20 mm to (106.3, 149.6)
- moved R2 0.13 mm to (106.6, 141.0)
- turned SW1 to 90 degrees
Routing:
- net VCC: track 0.00 -> 173.0 mm, vias 0 -> 6
- net /A1: track 0.00 -> 89.4 mm, vias 0 -> 2
- net GND: track 0.00 -> 86.0 mm, vias 0 -> 11
- net /RESET: track 0.00 -> 81.9 mm, vias 0 -> 3
- net /MOSI: track 0.00 -> 67.8 mm, vias 0 -> 4
- net /A0: track 0.00 -> 65.0 mm, vias 0 -> 2
- net /SCK: track 0.00 -> 49.2 mm, vias 0 -> 4
- net /MISO: track 0.00 -> 42.5 mm, vias 0 -> 3
- net Net-(IC1-Pad12): track 0.00 -> 31.9 mm, vias 0 -> 1
- net /TXD: track 0.00 -> 28.2 mm, vias 0 -> 1
- net /RXD: track 0.00 -> 27.9 mm, vias 0 -> 1
- net /A3: track 0.00 -> 20.8 mm, vias 0 -> 1
- net Net-(IC1-Pad32): track 0.00 -> 20.3 mm, vias 0 -> 2
- net Net-(IC1-Pad9): track 0.00 -> 17.7 mm, vias 0 -> 2
- net /A2: track 0.00 -> 13.7 mm, vias 0 -> 3
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Other:
- board text removed: "DTR"

Commit message: small layout updates - finish for first prototyp
Parts:
- moved R1 0.13 mm to (98.8, 140.2)
Connections:
- P7 pad 4: Net-(P7-Pad4) -> /TXD
- P7 pad 6: Net-(P7-Pad6) -> /RXD
Routing:
- net /TXD: track 28.2 -> 31.3 mm, vias 1 -> 2
- net /RXD: track 27.9 -> 30.6 mm, vias 1 -> 2
- net GND: track 86.0 -> 87.3 mm
- net /MISO: track 42.5 -> 41.7 mm
