File: RHS_3.sch (KiCad schematic (older format))
At the start: 68 parts, among them IC1 ATMEGA328P-A, IC2 CC1101, IC3 CC1101_Chip, J1 Glass Breakage Detector, J2 ANT, P4 ISP Bottom, P5 ISP Top, P6 FTDI, P7 ISP 10, Q1 Si2305CDS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

Commit message: fix 100p
Parts:
- C27: value 100n -> 100p; LCSC Part # C1525 -> C1546
Changed lines of the file:
@@
 P 9400 2350
 F 0 "C27" H 9492 2396 50  0000 L CNN
-F 1 "100n" H 9492 2305 50  0000 L CNN
+F 1 "100p" H 9492 2305 50  0000 L CNN
 F 2 "Capacitor_SMD:C_0402_1005Metric" H 9400 2350 50  0001 C CNN
 F 3 "~" H 9400 2350 50  0001 C CNN
-F 4 "C1525" H 9400 2350 50  0001 C CNN "LCSC Part #"
+F 4 "C1546" H 9400 2350 50  0001 C CNN "LCSC Part #"
 	1    9400 2350
 	1    0    0    -1
